File: parlaV0/parlaV0.kicad_sch (KiCad schematic)
At the start: 0 parts

Commit message: agregar borrador circuito
Parts:
- added C1: 220p, symbol Device:C
- added C2, C3: 470n, symbol Device:C_Polarized
- added C4: 100n, symbol Device:C
- added C5, C6: 220u, symbol Device:C_Polarized
- added C7: 100u, symbol Device:C_Polarized
- added LS1: Speaker, symbol Device:Speaker
- added R1: R, symbol Device:R
- added RV1: 10k, symbol Device:R_Potentiometer
- added U1: LM386, symbol Amplifier_Audio:LM386
- added V1: 6V, symbol Simulation_SPICE:VDC
Connections:
- new net: C1.1, C3.2, U1.3 (+)
- new net: C7.1, U1.7 (BYPASS)
- new net: C4.2, R1.1
- new net: C3.1, RV1.2
- new net: C2.1, U1.2 (-)
- new net: C6.1, U1.6 (V+), V1.1
- new net: C4.1, C5.1, U1.5
- new net: C5.2, LS1.1
- new net GND: C1.2, C2.2, C6.2, C7.2, LS1.2, R1.2, RV1.3, U1.4 (GND), V1.2
- new net Vin: RV1.1
- no-connect marks 0 -> 2
Other:
- company: (none) -> piruetas SpA
- title: (none) -> parla

Commit message: agregar footprints
Parts:
- added V2: 1, TerminalBlock_Phoenix:TerminalBlock_Phoenix_MPT-0,5-2-2.54_1x02_P2.54mm_Horizontal, symbol Simulation_SPICE:VSIN
- C1, C4: footprint (none) -> Capacitor_THT:C_Disc_D5.0mm_W2.5mm_P2.50mm
- C2, C3, C5, C6, C7: footprint (none) -> Capacitor_THT:CP_Radial_D4.0mm_P2.00mm
- LS1: value Speaker -> 8; footprint (none) -> TerminalBlock_Phoenix:TerminalBlock_Phoenix_MPT-0,5-2-2.54_1x02_P2.54mm_Horizontal
- R1: value R -> 10; footprint (none) -> Resistor_THT:R_Axial_DIN0309_L9.0mm_D3.2mm_P2.54mm_Vertical
- RV1: footprint (none) -> Potentiometer_THT:Potentiometer_Alps_RK09Y11_Single_Horizontal
- U1: footprint (none) -> Package_DIP:DIP-8_W7.62mm
- V1: value 6V -> 6; footprint (none) -> TerminalBlock_Phoenix:TerminalBlock_Phoenix_MPT-0,5-2-2.54_1x02_P2.54mm_Horizontal
Connections:
- net Vin: now also V2.1
- net +6V: now reaches C6.1, U1.6 (V+), V1.1
- net GND renamed 0
- net 0: now also V2.2
Other:
- moved on the sheet: V1

Commit message: agregar logo
Parts:
- RV1: footprint Potentiometer_THT:Potentiometer_Alps_RK09Y11_Single_Horizontal -> Potentiometer_THT:Potentiometer_Alps_RK097_Single_Horizontal
Changed lines of the file:
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@@
 		(on_board yes)
 		(dnp no)
-		(fields_autoplaced yes)
 		(property "Reference" "RV1"
 			(at 57.15 55.8799 0)
@@
 			)
 		)
-		(property "Footprint" "Potentiometer_THT:Potentiometer_Alps_RK09Y11_Single_Horizontal"
-			(at 59.69 57.15 0)
+		(property "Footprint" "Potentiometer_THT:Potentiometer_Alps_RK097_Single_Horizontal"
+			(at 55.118 106.934 0)
 			(effects
 				(font
