File: parlaV1/parlav1/parlav1.kicad_sch (KiCad schematic)
At the start: 13 parts, among them J1 Screw_Terminal_01x02, J2 Screw_Terminal_01x02, U1 LM386

Commit message: añadida parlaV1 by misaa
Parts:
- added D1: 1n4007, Diode_SMD:D_SOD-323, symbol Device:D
- added H1, H2: PAD, Connector_PinHeader_2.54mm:PinHeader_1x01_P2.54mm_Vertical, symbol Mechanical:MountingHole_Pad
- added H3, H4: M3, MountingHole:MountingHole_3.2mm_M3, symbol Mechanical:MountingHole
- C1: LCSC (none) -> C107145
- C2, C3: footprint Capacitor_SMD:CP_Elec_6.3x7.7 -> Capacitor_SMD:CP_Elec_4x5.4; LCSC (none) -> C22387960
- C4: LCSC (none) -> C49678
- C5, C6: footprint Capacitor_SMD:CP_Elec_6.3x7.7 -> Capacitor_SMD:CP_Elec_6.3x5.4; LCSC (none) -> C3345
- C7: footprint Capacitor_SMD:CP_Elec_6.3x7.7 -> Capacitor_SMD:CP_Elec_5x5.4; LCSC (none) -> C72473
- J1, J2: value Screw_Terminal_01x02 -> T_BLOCK_2; footprint TerminalBlock_Phoenix:TerminalBlock_Phoenix_PT-1,5-2-3.5-H_1x02_P3.50mm_Horizontal -> TerminalBlock:TerminalBlock_bornier-2_P5.08mm
- LS1: value 8 -> T_BLOCK_2; footprint TerminalBlock_Phoenix:TerminalBlock_Phoenix_MPT-0,5-2-2.54_1x02_P2.54mm_Horizontal -> TerminalBlock:TerminalBlock_bornier-2_P5.08mm
- POT1: renamed from RV1; value 10k -> T_BLOCK_3; footprint TerminalBlock_Phoenix:TerminalBlock_Phoenix_PT-1,5-3-3.5-H_1x03_P3.50mm_Horizontal -> Connector_PinHeader_2.54mm:PinHeader_1x03_P2.54mm_Vertical
- R1: footprint Resistor_SMD:R_1206_3216Metric -> Resistor_SMD:R_0805_2012Metric; LCSC (none) -> C2907296
- U1: footprint Package_DIP:DIP-8_W7.62mm -> Package_DIP:DIP-8_W7.62mm_LongPads
Connections:
- net GND: now also POT1.1; no longer POT1.3
- net Vin: now also POT1.3; no longer POT1.1
- net at U1.1 (GAIN): now also H1.1
- net at U1.8 (GAIN): now also H2.1
- net +6V renamed VCC
- net VCC: now also D1.1 (K); no longer J2.1 (Pin_1)
- new net: D1.2 (A), J2.1 (Pin_1)
- no-connect marks 2 -> 0
Other:
- note added: "dc in 5 - 12v"
- note added: "input"
- note added: "pot 10k"
- note added: "speaker out 8 ohm"
- moved on the sheet: J2
