File: parla-v0-revB/parla-v0-revB.kicad_sch (KiCad schematic)
At the start: 16 parts, among them J1 AudioJack2_SwitchT, J2 AudioJack2_SwitchT, J3 AudioJack2_SwitchT, J4 AudioJack2_SwitchT, U1 PAM8403D

Commit message: actualizada version smd
Parts:
- added C10: 100n, Capacitor_SMD:C_0805_2012Metric_Pad1.18x1.45mm_HandSolder, symbol Device:C
- added C4, C5, C6: 1u, Capacitor_SMD:C_0805_2012Metric_Pad1.18x1.45mm_HandSolder, symbol Device:C
- added C7: 100u, Capacitor_SMD:CP_Elec_6.3x7.7, symbol Device:C_Polarized
- added C8: 220u, Capacitor_SMD:CP_Elec_6.3x5.4, symbol Device:C_Polarized
- added C9: 10u, Capacitor_SMD:CP_Elec_4x5.4, symbol Device:C_Polarized
- added D1: 1N4007, Diode_SMD:D_SOD-323_HandSoldering, symbol Diode:1N4007
- added D8: LED, LED_THT:LED_D5.0mm, symbol Device:LED
- added J5: Barrel_Jack_Switch, Connector_BarrelJack:BarrelJack_Horizontal, symbol Connector:Barrel_Jack_Switch
- added R5: 1k, Resistor_SMD:R_0805_2012Metric_Pad1.20x1.40mm_HandSolder, symbol Device:R
- added SW3: SW_SPDT, dis8644:spdt_ssd12d00g3, symbol Switch:SW_SPDT
- added U2: L7805, Package_TO_SOT_SMD:TO-252-2, symbol Regulator_Linear:L7805
- C1, C2: footprint (none) -> Capacitor_SMD:C_Elec_4x5.4; LCSC (none) -> C2895732
- C3: footprint (none) -> Capacitor_SMD:C_0805_2012Metric_Pad1.18x1.45mm_HandSolder; LCSC (none) -> C49678
- J1, J2, J3, J4: footprint (none) -> dis8644:PJ301M-12-T_TN_S
- R3, R4: footprint (none) -> Resistor_SMD:R_0805_2012Metric_Pad1.20x1.40mm_HandSolder; LCSC (none) -> C17414
- RV1, RV2: footprint (none) -> Potentiometer_THT:Potentiometer_Bourns_PTV09A-1_Single_Vertical
- U1: LCSC (none) -> C5122557
Connections:
- net +5V: now also C10.1, C4.2, C5.2, C6.2, C8.1, C9.1, D8.2 (A), U2.3 (OUT)
- net GND: now also C10.2, C4.1, C5.1, C6.1, C7.2, C8.2, C9.2, J5.2, R5.1, U2.2 (GND)
- new net: D8.1 (K), R5.2
- new net: J5.1, SW3.1 (A)
- new net: D1.2 (A), SW3.2 (B)
- new net +12V: C7.1, D1.1 (K), U2.1 (IN)
- no-connect marks 6 -> 8
Other:
- note added: "ALIMENTACIÓN"
- note added: "FUENTES ENTRE 7 y 12V Centro positivo"
- note added: "PIN 3 = 12v PIN 2 = 5v PIN 1 = GND"
- note added: "TODOS LOS CHIPS DEBEN SER ALIMENTADOS CON 5V"
