File: parla-guitarra-v-0/parla-guitarra-v-0.kicad_sch (KiCad schematic)
At the start: 7 parts, among them J1 AudioJack2_SwitchT, U1 LM386

Commit message: agregar borrador
Parts:
- removed C1: 470n, symbol Device:C
- added C5: 47u, symbol Device:C_Polarized
- added C6: 200n, symbol Device:C
- added J2: Screw_Terminal_01x02, symbol Connector:Screw_Terminal_01x02
- added RV1: 5k, symbol Device:R_Potentiometer
Connections:
- net GND: now also C5.2, C6.2, J2.2 (Pin_2)
- net at C2.1, U1.3 (+): no longer J1.3
- net at U1.2 (-): now also J1.3
- net at U1.1 (GAIN): now also RV1.1; no longer U1.8 (GAIN)
- net +5V renamed +9V
- net +9V: now also C5.1, C6.1, J2.1 (Pin_1)
- new net: RV1.2, RV1.3, U1.8 (GAIN)
Other:
- note removed: "1 a 8 smokey amp"
- title: (none) -> parla-guitarra
