File: parla-linea-extensor/parla-linea-extensor-v-0-rev-a/parla-linea-extensor-v-0-rev-a.kicad_sch (KiCad schematic)
At the start: 0 parts

Commit message: agregar mas sobre parla linea extensor
Parts:
- added J1: AudioJack3_SwitchT, symbol Connector_Audio:AudioJack3_SwitchT
- added LS1: Speaker, TerminalBlock:TerminalBlock_MaiXu_MX126-5.0-02P_1x02_P5.00mm, symbol Device:Speaker
Connections:
- new net: J1.T, LS1.1
- new net: J1.R, LS1.2
- no-connect marks 0 -> 1
Other:
- note added: "este producto es un extensor de parla linea"
- note added: "pam8403 emite salida de R en positivo y negativo"
- note added: "pregunta como hacer que funcione con cables TRS y TS"
- company: (none) -> piruetas SpA
- title: (none) -> parla linea extensor v0
