File: parla-linea/parla-linea-v-0-rev-a/parla-linea-v-0-rev-a.kicad_pcb (KiCad board)
At the start: 0 parts

Commit message: trazado
Parts:
- added C1: C, parla-linea-v-0-rev-a:C0805, F.Cu at (64.0, 86.0)
- added C2: 100n, parla-linea-v-0-rev-a:C0805, F.Cu at (81.0, 82.0)
- added C3: 100u, parla-linea-v-0-rev-a:CAP-SMD_BD6.3-L6.6-W6.6-LS7.6-FD, F.Cu at (63.6, 64.5)
- added C4: 10u, parla-linea-v-0-rev-a:CAP-SMD_BD4.0-L4.3-W4.3-FD, F.Cu at (66.0, 72.7)
- added C6: C, parla-linea-v-0-rev-a:C0805, F.Cu at (62.0, 91.0)
- added C7: 100n, parla-linea-v-0-rev-a:C0805, F.Cu at (75.0, 82.0)
- added D1: 1N4007, parla-linea-v-0-rev-a:SOD-323_L1.8-W1.3-LS2.5-RD, F.Cu at (58.0, 61.0)
- added D2: LED, Eurocad:LED3mm, F.Cu at (87.0, 55.3)
- added H1: M3, MountingHole:MountingHole_3.2mm_M3, F.Cu at (55.0, 55.0)
- added H2: M3, MountingHole:MountingHole_3.2mm_M3, F.Cu at (95.0, 55.0)
- added H3: M3, MountingHole:MountingHole_3.2mm_M3, F.Cu at (55.0, 95.0)
- added H4: M3, MountingHole:MountingHole_3.2mm_M3, F.Cu at (95.0, 95.0)
- added J1: AudioJack2_SwitchT, Connector_Audio:Jack_3.5mm_QingPu_WQP-PJ398SM_Vertical_CircularHoles, F.Cu at (86.3, 69.8)
- added J2: AudioJack2_SwitchT, Connector_Audio:Jack_3.5mm_QingPu_WQP-PJ398SM_Vertical_CircularHoles, F.Cu at (86.3, 80.5)
- added J3: Screw_Terminal_01x02, TerminalBlock:TerminalBlock_MaiXu_MX126-5.0-02P_1x02_P5.00mm, F.Cu at (67.6, 55.1)
- added J4: Conn_01x01, Connector_Wire:SolderWire-0.25sqmm_1x01_D0.65mm_OD1.7mm, F.Cu at (53.1, 64.5)
- added J5: Screw_Terminal_01x02, TerminalBlock:TerminalBlock_MaiXu_MX126-5.0-02P_1x02_P5.00mm, F.Cu at (80.0, 54.9)
- added J6: AudioJack3_SwitchTR, Connector_Audio:Jack_3.5mm_CUI_SJ1-3525N_Horizontal, F.Cu at (54.5, 75.0)
- added J7: Conn_01x03_Pin, Connector_PinHeader_2.54mm:PinHeader_1x03_P2.54mm_Vertical, F.Cu at (53.5, 86.0)
- added R1: 10k, parla-linea-v-0-rev-a:R0805, F.Cu at (64.0, 79.0)
- added R2: 10k, parla-linea-v-0-rev-a:R0805, F.Cu at (67.0, 79.0)
- added R3: 1k, parla-linea-v-0-rev-a:R0805, F.Cu at (87.0, 61.0)
- added RV1: 100kB, Potentiometer_THT:Potentiometer_Alps_RK163_Dual_Horizontal, F.Cu at (70.0, 94.8)
- added U1: PAM8403D, parla-linea-v-0-rev-a:SOP-16_L10.0-W3.9-P1.27-LS6.0-BL, F.Cu at (75.0, 75.0)
- added U2: L7805, parla-linea-v-0-rev-a:TO-252-2_L6.6-W6.1-P4.57-LS9.9-BR-CW, F.Cu at (74.6, 65.0)
Routing:
- net +5V: track 0.00 -> 59.7 mm
- net Net-(U1-LOUT+): track 0.00 -> 48.6 mm, vias 0 -> 1
- net Net-(U1-ROUT+): track 0.00 -> 32.0 mm, vias 0 -> 2
- net Net-(U1-INR): track 0.00 -> 31.0 mm, vias 0 -> 1
- net Net-(U1-INL): track 0.00 -> 29.3 mm
- net Net-(U1-LOUT-): track 0.00 -> 22.5 mm, vias 0 -> 2
- net Net-(J7-Pin_2): track 0.00 -> 21.2 mm, vias 0 -> 1
- net Net-(U1-ROUT-): track 0.00 -> 20.6 mm, vias 0 -> 2
- net Net-(C6-Pad2): track 0.00 -> 19.7 mm, vias 0 -> 1
- net Net-(C1-Pad2): track 0.00 -> 19.2 mm
- net Net-(D1-K): track 0.00 -> 13.7 mm
- net Net-(J6-PadR): track 0.00 -> 12.3 mm
- net +9V: track 0.00 -> 11.6 mm
- net Net-(J7-Pin_3): track 0.00 -> 10.9 mm
- net Net-(J7-Pin_1): track 0.00 -> 10.6 mm
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- added copper zone on B.Cu, net GND
- added copper zone on F.Cu, net GND
Other:
- board outline added: 50 x 50 mm
- copper layers 0 -> 2
- board text added: "L"
- board text added: "R"
- board text added: "gnd"
- board text added: "stereo"
- board text added: "sum L+R"

Commit message: agregar pcba
Parts:
- C1, C6: value C -> 1u
Other:
- board text added: "2026-10"
- board text added: "parla-linea"
- board text added: "rev-a"
- board text added: "v0"
